Commit message: feat: Full RL training pipeline — 4 tasks, rewards, domain randomization, local launcher
- Add SO-100 linear rail URDF (so100_rail.urdf) with wrist camera link
- Update P2S printer URDF: door hinge origin fix, joint limit corrections, door handle marker
- Rename mesh files from hyphens to underscores (X_axis_nozzle_1, Y_axis_1, Z_bed_1)
- Rewrite scene_cfg.py: rail actuator, FrameTransformer for door handle, staging area
- Implement 4 task environments: OpenDoor, PickPrint, PlacePrint, CloseDoor
- Add 13 reward functions and 6 termination conditions
- Add domain randomization (door stiffness, object mass, friction, lighting)
- Add PPO configs for all tasks including FullCycle
- Register 4 gym environments (PrinterArm-*-v0)
- Create local training scripts and run_full_cycle.py state machine
- Delete old sim/isaac_lab/tasks/ (superseded by printer_arm_tasks/)

Co-Authored-By: Claude Opus 4.6 <noreply@anthropic.com>

File: sim/isaac_lab/assets/p2s/urdf/BAMBULAB_P2S.xacro (robot description, xacro)
@@ -86,10 +86,10 @@
 <link name="Door_1">
   <inertial>
-    <origin xyz="0.08303570031679738 -0.02685731793471252 -0.06313292896757283" rpy="0 0 0"/>
+    <origin xyz="0.03 -0.03 0" rpy="0 0 0"/>
     <mass value="1.8912702022608048"/>
     <inertia ixx="0.02213" iyy="0.03801" izz="0.015883" ixy="2.6e-05" iyz="3e-06" ixz="-8.5e-05"/>
   </inertial>
   <visual>
-    <origin xyz="-0.13216 -0.080867 -0.348717" rpy="0 0 0"/>
+    <origin xyz="0.03 -0.03 0" rpy="0 0 0"/>
     <geometry>
       <mesh filename="package://BAMBULAB_P2S_description/meshes/Door_1.stl" scale="0.001 0.001 0.001"/>
@@ -98,5 +98,5 @@
   </visual>
   <collision>
-    <origin xyz="-0.13216 -0.080867 -0.348717" rpy="0 0 0"/>
+    <origin xyz="0.03 -0.03 0" rpy="0 0 0"/>
     <geometry>
       <mesh filename="package://BAMBULAB_P2S_description/meshes/Door_1.stl" scale="0.001 0.001 0.001"/>
@@ -126,5 +126,5 @@
 </joint>
 <joint name="Revolute 8" type="revolute">
-  <origin xyz="0.13216 0.080867 0.348717" rpy="0 0 0"/>
+  <origin xyz="-0.03 0.03 0" rpy="0 0 0"/>
   <parent link="base_link"/>
   <child link="Door_1"/>

File: sim/isaac_lab/assets/p2s/urdf/p2s_printer.urdf (robot description, URDF)
Before this commit: robot BAMBULAB_P2S, 5 links, 4 joints
Links:
- removed link X-axis_nozzle_1
- removed link Y-axis_1
- removed link Z-bed_1
- added link X_axis_nozzle_1, mass 0.675060661578604; collision mesh filename=../meshes/X_axis_nozzle_1.stl scale=0.001 0.001 0.001; visual mesh filename=../meshes/X_axis_nozzle_1.stl scale=0.001 0.001 0.001
- added link Y_axis_1, mass 1.2845247547395635; collision mesh filename=../meshes/Y_axis_1.stl scale=0.001 0.001 0.001; visual mesh filename=../meshes/Y_axis_1.stl scale=0.001 0.001 0.001
- added link Z_bed_1, mass 10.019848039853946; collision mesh filename=../meshes/Z_bed_1.stl scale=0.001 0.001 0.001; visual mesh filename=../meshes/Z_bed_1.stl scale=0.001 0.001 0.001
- added link door_handle_marker, mass 0.001; visual box size=0.04 0.04 0.001
Joints:
- removed joint X-axis
- removed joint Y-axis
- removed joint Z-axis
- added joint X_axis: type prismatic, parent Y_axis_1, child X_axis_nozzle_1, origin xyz=-0.06258 -0.057764 -0.053445 rpy=0 0 0, axis -1.0 0.0 0.0, limit lower=-0.21 upper=0.0 effort=100 velocity=100
- added joint Y_axis: type prismatic, parent base_link, child Y_axis_1, origin xyz=0.15016 0.450867 0.554722 rpy=0 0 0, axis 0.0 1.0 0.0, limit lower=-0.25 upper=0.0 effort=100 velocity=100
- added joint Z_axis: type prismatic, parent base_link, child Z_bed_1, origin xyz=0.126543 0.173367 0.157117 rpy=0 0 0, axis 0.0 0.0 -1.0, limit lower=-0.31 upper=0.0 effort=100 velocity=100
- added joint marker_joint: type fixed, parent Door_1, child door_handle_marker, origin xyz=0.15 -0.03 -0.05 rpy=0 0 0
- joint door_hinge: origin xyz=0.13216 0.080867 0.348717 rpy=0 0 0 -> xyz=-0.03 0.03 0 rpy=0 0 0
