Commit message: feat: scene composition fixes — printer alignment, lights, wrist cam, materials
- Printer: positioned so volume center sits at world (0, 0.4, 0); door
  uses glass material, body switched to gray; build_plate and print_object
  re-aligned to Z_bed_1 surface
- Robot: rail axis flipped to X (world X range 0~0.6); base at (0.3, 0, 0)
  with Z-axis 180° rotation; arm actuators boosted (effort 80, stiff 2000)
  so arm reliably holds pose against gravity
- WOWROBO Wrist_Cam_Mount.stl integrated on gripper; gripper_camera_link
  parented to gripper with visually-calibrated origin (xyz -0.0 -0.0 -0.07,
  rpy -0.4 0 0); so100.urdf and so100_rail.urdf kept in sync
- Scene viewer (load_scene_standalone) calls so100_utils.attach_wrist_camera
  shared helper; load_so100_standalone also wired up
- RL env _PrinterArmBase now applies PBR material binding to printer prims
  (gray/glass/brown/red) so RL viewport renders correctly
- DomeLight + DistantLight added for ambient illumination; interior
  SphereLights mounted via URDF light_l/r_link so they follow the printer
- Stepper-bed semantics: Z_axis drive holds position (stiff 100k); Z_bed_1
  link gravity disabled in viewer; door_hinge max_force=0 for free swing
- run_sim.sh: --enable_cameras propagated to all modes; --load-urdf and
  --load-scene now compatible with --display

Co-Authored-By: Claude Opus 4.7 <noreply@anthropic.com>

File: sim/isaac_lab/assets/p2s/urdf/p2s_printer.urdf (robot description, URDF)
Before this commit: robot BAMBULAB_P2S, 6 links, 5 joints
Links:
- added link light_l_link, mass 0.001
- added link light_r_link, mass 0.001
- link door_handle_marker: geometry visual box size=0.05 0.05 0.002
Joints:
- added joint light_l_joint: type fixed, parent base_link, child light_l_link, origin xyz=-0.04 0.10 0.45 rpy=0 0 0
- added joint light_r_joint: type fixed, parent base_link, child light_r_link, origin xyz=0.31 0.10 0.45 rpy=0 0 0

File: sim/isaac_lab/assets/so100/so100.urdf (robot description, URDF)
Before this commit: robot so_arm100, 7 links, 6 joints
Links:
- added link gripper_camera_link, mass 0.01; visual box size=0.025 0.025 0.001
- link gripper: geometry visual mesh filename=assets/Fixed_Jaw_Motor.stl; visual mesh filename=assets/Wrist_Cam_Mount.stl
Joints:
- added joint wrist_camera_joint: type fixed, parent gripper, child gripper_camera_link, origin xyz=-0.003 0.003 -0.073 rpy=-2.0 0.0 0.0

File: sim/isaac_lab/assets/so100/so100_rail.urdf (robot description, URDF)
Before this commit: robot so_arm100_rail, 9 links, 8 joints
Links:
- removed link wrist_camera_link
- added link gripper_camera_link, mass 0.01; visual box size=0.025 0.025 0.015
- link gripper: geometry visual mesh filename=assets/Fixed_Jaw_Motor.stl; visual mesh filename=assets/Wrist_Cam_Mount.stl
- link rail_base: geometry collision box size=0.6 0.08 0.02; visual box size=0.6 0.08 0.02
Joints:
- joint rail_slide: axis 0 1 0 -> 1 0 0
- joint wrist_camera_joint: child wrist_camera_link -> gripper_camera_link; origin xyz=0.0 -0.04 0.015 rpy=0 0.52 0 -> xyz=0.0 -0.0 -0.07 rpy=-0.4 0.0 0.0
