Commit message: feat: inspect mode + wrist camera calibration
- New inspect_rl_env.py: spawns the same scene_cfg env (PrinterArm-OpenDoor-v0)
  with zero-action loop, no PPO. Wired via run_sim.sh --inspect for fast
  manual scene tuning.
- run_sim.sh: --display now calls xhost +local:docker so the container
  can reach the host X server (was failing with IWindowing error).
- Wrist camera transform calibrated visually in inspect viewer
  (translate (0, -0.02, 0), rotate XYZ (-110°, 0°, 0°)): applied as
  CameraCfg.offset for RL and in so100_utils.attach_wrist_camera for
  standalone viewers. Box visual now has explicit <origin> in URDF so
  shape/pose match URDF Preview.

Co-Authored-By: Claude Opus 4.7 <noreply@anthropic.com>

File: sim/isaac_lab/assets/so100/so100.urdf (robot description, URDF)
Before this commit: robot so_arm100, 8 links, 7 joints
Links:
- link gripper_camera_link: geometry visual box size=0.025 0.025 0.015
Joints:
- joint wrist_camera_joint: origin xyz=-0.003 0.003 -0.073 rpy=-2.0 0.0 0.0 -> xyz=-0.003 0.003 -0.073 rpy=-0.4 0.0 0.0

File: sim/isaac_lab/assets/so100/so100_rail.urdf (robot description, URDF)
Before this commit: robot so_arm100_rail, 9 links, 8 joints
Joints:
- joint wrist_camera_joint: origin xyz=0.0 -0.0 -0.07 rpy=-0.4 0.0 0.0 -> xyz=-0.003 0.003 -0.073 rpy=-0.4 0.0 0.0
